File: Nanopositioner/Electronics/nanopositioner_driver_v1.kicad_sch (KiCad schematic)
At the start: 75 parts, among them J3 DE9_Pins, Q1 MJD45H11T4G, Q2 MJD44H11T4G, Q3 MJD45H11T4G, Q4 MJD44H11T4G, Q5 MJD45H11T4G, Q6 MJD44H11T4G, Q7 MJD44H11T4G, Q8 MJD45H11T4G, Q9 BCX56, SW1 NRST, U1 ISO7720D, U2 DAC8552, U3 DAC8552, U4 STM32G431CBTx, U5 OPA552U, U6 ISO7720D, U7 OPA552U, U8 OPA552U, U9 OPA552U, Y1 8MHz

Commit message: Updated the design of the mainboard
Parts:
- added C18, C19, C20, C29, C31, C39: 10u, symbol Device:C_Small
- added C30, C32: 100n, symbol Device:C_Small
- added D2: BZT52-C5V6, Diode_SMD:D_SOD-123F, symbol Diode:BZT52Bxx
- added D3, D4, D5, D6: LED_Small, symbol Device:LED_Small
- added J1, J2, J4: DE9_Pins, symbol Connector:DE9_Pins
- added J5: USB_C_Receptacle_USB2.0_16P, symbol Connector:USB_C_Receptacle_USB2.0_16P
- added JP3: 6V2_TEST, symbol Jumper:Jumper_2_Small_Open
- added NT4, NT5, NT6, NT7: NetTie_2, symbol Device:NetTie_2
- added Q10: BCX56, symbol Simulation_SPICE:NPN
- added R18: 20k, symbol Device:R_Small_US
- added R19, R20, R21, R22: 1k, symbol Device:R_Small_US
- added U10: REF5050AD, Package_SO:SOIC-8_3.9x4.9mm_P1.27mm, symbol Reference_Voltage:REF5050AD
- added U11: CH340C, Package_SO:SOIC-16_3.9x9.9mm_P1.27mm, symbol Interface_USB:CH340C
Connections:
- net CONN_TEST_0 is gone; now on net CONN_TEST_1_P: J3.4
- net CONN_TEST_1 is gone; now on net PIEZO_CH1_PA: J3.5
- net +3V3: now also U1.1 (VCC1), U6.1 (VCC1)
- net +5V_HV: now also U2.1 (V_{DD}), U3.1 (V_{DD}), C30.2, C31.2, C32.2, C39.2
- net +60V: now also Q10.1 (C), R18.1
- net GND: now also J3.1, C30.1, C31.1, C32.1, C39.1, D3.1 (K), D4.1 (K), D5.1 (K), D6.1 (K), J1.1, J2.1, J4.1
- net GNDV: now also C18.1, C19.1, C20.1, C29.1, D2.2 (A), U10.4 (GND)
- net PIEZO_CH1_PA: no longer J3.9
- net PIEZO_CH2_PA: now also J1.5; no longer J3.8
- net PIEZO_CH3_PA: now also J2.5; no longer J3.7
- net PIEZO_CH4_PA: now also J4.5; no longer J3.6
- net ~{CS4}: now reaches U4.17 (PB1)
- net ~{CS4}: now also J4.8
- net ~{CS3}: now reaches U4.18 (PB2)
- net ~{CS3}: now also J2.8
- net ~{CS2}: now reaches U4.25 (PB11)
- net ~{CS2}: now also J1.8
- net ~{CS1}: now reaches U4.26 (PB12)
- net ~{CS1}: now also J3.8
- net CLK1_2: now reaches U4.27 (PB13)
- net CLK1_2: now also J3.3, J1.3
- net DO1: now reaches U4.28 (PB14)
- net DO1: now also J3.7, NT5.2
- net DIN1: now reaches U4.29 (PB15)
- net DIN1: now also J3.2, NT4.2
- net CONN_TEST_1_P: now reaches U4.30 (PA8)
- net CONN_TEST_1_P: now also R22.1
- net CONN_TEST_2_P: now reaches U4.31 (PA9)
- net CONN_TEST_2_P: now also J1.4, R21.1
- net CONN_TEST_3_P: now reaches U4.32 (PA10)
- net CONN_TEST_3_P: now also J2.4, R20.1
- net CONN_TEST_4_P: now reaches U4.33 (PA11)
- net CONN_TEST_4_P: now also J4.4, R19.1
- net CLK3_4: now reaches U4.40 (PB3)
- net CLK3_4: now also J2.3, J4.3
- net DO3: now reaches U4.41 (PB4)
- net DO3: now also J2.7, NT6.2
- net DIN3: now reaches U4.42 (PB5)
- net DIN3: now also J2.2, NT7.2
- net UART1_TX: now reaches U4.43 (PB6)
- net UART1_TX: now also U11.3 (RXD)
- net UART1_RX: now reaches U4.44 (PB7)
- net UART1_RX: now also U11.2 (TXD)
- net +5V_REF: now reaches U2.2 (V_{REF})
- net +5V_REF: now also U3.2 (V_{REF}), C20.2, C29.2, U10.6 (Vout)
- new net: D5.2 (A), R21.2
- new net: D4.2 (A), R20.2
- new net: D3.2 (A), R19.2
- new net: D2.1 (K), Q10.2 (B), R18.2
- new net: JP3.1 (A), Q10.3 (E)
- new net: C19.2, JP3.2 (B), U10.2 (Vin)
- new net: D6.2 (A), R22.2
- new net: C18.2, U10.5 (Trim/NR)
- new net: J5.A1 (GND), J5.A12 (GND), J5.B1 (GND), J5.B12 (GND)
- new net: J5.A4 (VBUS), J5.A9 (VBUS), J5.B4 (VBUS), J5.B9 (VBUS)
- new net +5V: J1.6, J2.6, J3.6, J4.6
- new net DIN2: J1.2, NT4.1
- new net DIN4: J4.2, NT7.1
- new net DO2: J1.7, NT5.1
- new net DO4: J4.7, NT6.1
- no-connect marks 4 -> 9
Other:
- note added: "CH1"
- note added: "CH2"
- note added: "CH3"
- note added: "CH4"
- note added: "For connection detection, CONN_TEST_x_P will go to 5V when the piezo stage is connected"
- note removed: "For connection detection, CONN_TEST_0 and 1 are shorted when piezo stage is connected"
- moved on the sheet: C1, C10, C11, C12, C13, C14, C15, C16, C17, C2, C21, C22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

Commit message: Updated driver design
Parts:
- removed J5: USB_C_Receptacle_USB2.0_16P, symbol Connector:USB_C_Receptacle_USB2.0_16P
- removed NT1, NT3: VDDA, symbol Device:NetTie_2
- added C40, C41, C43: 100n, Capacitor_SMD:C_0805_2012Metric, symbol Device:C_Small
- added C42: 220u 100V, Capacitor_THT:CP_Radial_D13.0mm_P5.00mm, symbol Device:C_Polarized_Small_US
- added C44, C45: 10u, Capacitor_SMD:C_0805_2012Metric, symbol Device:C_Small
- added D7: SS310, Diode_SMD:D_SMB, symbol Device:D_Schottky_Small
- added D8: BZT52-B75, Diode_SMD:D_SOD-123F, symbol Diode:BZT52Bxx
- added D9: OVP_INDICATOR, Connector_JST:JST_XH_B2B-XH-A_1x02_P2.50mm_Vertical, symbol Device:LED_Small
- added H1, H2, H3, H4, H5: MountingHole, MountingHole:MountingHole_3.2mm_M3, symbol Mechanical:MountingHole
- added J10: Conn_02x08_Odd_Even, Connector_PinHeader_2.54mm:PinHeader_2x08_P2.54mm_Vertical, symbol Connector_Generic:Conn_02x08_Odd_Even
- added J5: HV_IN, TerminalBlock:TerminalBlock_bornier-2_P5.08mm, symbol Connector_Generic:Conn_01x02
- added J6: USB_UART_RECEPTACLE, SamacSys_Parts:GCT_USB4105GFA120, symbol Connector:USB_C_Receptacle_USB2.0
- added J8: SWD, Connector_PinSocket_2.54mm:PinSocket_1x04_P2.54mm_Vertical, symbol Connector_Generic:Conn_01x04
- added Q11, Q12: NCE1540K, symbol Simulation_SPICE:PMOS
- added R23: 10M, Capacitor_SMD:C_0805_2012Metric, symbol Device:R_Small_US
- added R24, R27: 100k, Capacitor_SMD:C_0805_2012Metric, symbol Device:R_Small_US
- added R25, R26: 5k49, Capacitor_SMD:C_0805_2012Metric, symbol Device:R_Small_US
- added RV1: 1M, Capacitor_SMD:C_0805_2012Metric, symbol Device:R_Potentiometer_US
- added U12: AMS1117-3.3, Package_TO_SOT_SMD:SOT-223-3_TabPin2, symbol Regulator_Linear:AMS1117-3.3
- C1, C2: footprint (none) -> Capacitor_SMD:C_0603_1608Metric
- C10, C11, C12, C13, C18, C19, C20, C21, C29, C3, C30, C31, C32, C33, C35, C37, C39, C4, C7, C8, C9, R1, R10, R11, R12, R13, R14, R15, R16, R17, R18, R19, R2, R20, R21, R22, R3, R4, R5, R6, R7, R8, R9: footprint (none) -> Capacitor_SMD:C_0805_2012Metric
- C14, C16, C17, C22, C24, C25, C27, C28, C34, C36, C38, C6: footprint (none) -> Capacitor_SMD:C_1206_3216Metric
- C15, C23, C26, C5: footprint (none) -> Capacitor_THT:CP_Radial_D13.0mm_P5.00mm
- D3, D4, D5, D6: footprint (none) -> Connector_JST:JST_XH_B2B-XH-A_1x02_P2.50mm_Vertical
- J1, J2, J3, J4: footprint (none) -> Connector_Dsub:DSUB-9_Socket_Horizontal_P2.77x2.84mm_EdgePinOffset7.70mm_Housed_MountingHolesOffset9.12mm
- JP1: footprint (none) -> Connector_PinHeader_2.54mm:PinHeader_1x02_P2.54mm_Vertical
- JP2, JP3: footprint (none) -> Jumper:SolderJumper-2_P1.3mm_Open_Pad1.0x1.5mm
- NT2, NT4, NT5, NT6, NT7: footprint (none) -> NetTie:NetTie-2_SMD_Pad2.0mm
- SW1: footprint (none) -> SamacSys_Parts:TL3342F260QG
- Y1: footprint (none) -> SamacSys_Parts:YSX530
Connections:
- net +3V3: now also C10.2, C11.2, C12.2, C21.2, C3.2, C4.2, C9.2, U11.16 (VCC), U11.4 (V3), U4.1 (VBAT), U4.21 (VDDA), U4.24 (VDD), U4.36 (VDD), U4.48 (VDD), C41.2, C43.1, C44.2, J10.10 (Pin_10), J8.1 (Pin_1), U12.2 (VO)
- net +5V: now also C40.2, C45.2, J10.12 (Pin_12), J6.A4 (VBUS), J6.A9 (VBUS), J6.B4 (VBUS), J6.B9 (VBUS), U12.3 (VI)
- net +60V: now also C42.1, Q11.1 (D)
- net GND: now also U11.1 (GND), C40.1, C41.1, C43.2, C44.1, C45.1, J10.14 (Pin_14), J10.16 (Pin_16), J6.A1 (GND), J6.A12 (GND), J6.B1 (GND), J6.B12 (GND), J6.S1 (SHIELD), J8.4 (Pin_4), R25.1, R26.1, U12.1 (GND)
- net GNDV: now also J1.9, J2.9, J3.9, J4.9, C42.2, D7.2 (A), D8.2 (A), D9.1 (K), J5.2 (Pin_2), R23.2, R24.1
- net VDD: no longer C10.2, C11.2, C12.2, C21.2, C9.2, U4.1 (VBAT), U4.24 (VDD), U4.36 (VDD), U4.48 (VDD)
- net VDDA: no longer C3.2, C4.2, U4.21 (VDDA)
- net UART2_TX: now reaches U4.10 (PA2)
- net UART2_TX: now also J10.13 (Pin_13)
- net UART2_RX: now reaches U4.11 (PA3)
- net UART2_RX: now also J10.15 (Pin_15)
- net PB0: now reaches U4.16 (PB0)
- net PB0: now also J10.8 (Pin_8)
- net PC13: now reaches U4.2 (PC13)
- net PC13: now also J10.2 (Pin_2)
- net BTN3: now reaches U4.22 (PB10)
- net BTN3: now also J10.5 (Pin_5)
- net PC14: now reaches U4.3 (PC14)
- net PC14: now also J10.4 (Pin_4)
- net BTN1: now reaches U4.34 (PA12)
- net BTN1: now also J10.1 (Pin_1)
- net SWDIO: now reaches U4.37 (PA13)
- net SWDIO: now also J8.2 (Pin_2)
- net SWCLK: now reaches U4.38 (PA14)
- net SWCLK: now also J8.3 (Pin_3)
- net BTN4: now reaches U4.39 (PA15)
- net BTN4: now also J10.7 (Pin_7)
- net PC15: now reaches U4.4 (PC15)
- net PC15: now also J10.6 (Pin_6)
- net BTN2: now reaches U4.46 (PB9)
- net BTN2: now also J10.3 (Pin_3)
- net BTN5: now reaches U4.8 (PA0)
- net BTN5: now also J10.9 (Pin_9)
- net BTN6: now reaches U4.9 (PA1)
- net BTN6: now also J10.11 (Pin_11)
- net USB_DP: now reaches U11.5 (UD+)
- net USB_DP: now also J6.A6 (D+), J6.B6 (D+)
- net USB_DN: now reaches U11.6 (UD-)
- net USB_DN: now also J6.A7 (D-), J6.B7 (D-)
- new net: Q11.2 (G), Q12.3 (S)
- new net: J6.B5 (CC2), R26.2
- new net: J6.A5 (CC1), R25.2
- new net: D9.2 (A), R27.1
- new net: Q12.1 (D), R24.2, R27.2
- new net: D8.1 (K), Q12.2 (G), R23.1, RV1.3
- new net +60V_IN: D7.1 (K), J5.1 (Pin_1), Q11.3 (S), RV1.1, RV1.2
- no-connect marks 9 -> 14
Other:
- note added: "IO"
- note added: "LV Regulators & Input Protection"
- note added: "Maximum Vin at 150V"
- note added: "Microcontroller"
- note added: "OVP Protection"
- note added: "VDD"
- note added: "VDDA"
- moved on the sheet: C1, C10, C11, C12, C13, C14, C15, C16, C17, C18, C19, C2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

Commit message: Updated the complete PCB design
Parts:
- removed NT2: VDDA, NetTie:NetTie-2_SMD_Pad2.0mm, symbol Device:NetTie_2
- removed NT4, NT5, NT6, NT7: NetTie_2, NetTie:NetTie-2_SMD_Pad2.0mm, symbol Device:NetTie_2
- removed Q7: MJD44H11T4G, symbol Simulation_SPICE:NPN
- removed Q8: MJD45H11T4G, symbol Simulation_SPICE:PNP
- removed R17, R18: 20k, Capacitor_SMD:C_0805_2012Metric, symbol Device:R_Small_US
- added C46, C47, C48, C49: 100n, Capacitor_SMD:C_0805_2012Metric, symbol Device:C_Small
- added C50, C53, C55, C57: 220p 100V, Capacitor_SMD:C_1206_3216Metric, symbol Device:C_Small
- added C51, C52, C54, C56: C_CAP, Capacitor_SMD:C_0805_2012Metric, symbol Device:C_Small
- added D10: PIEZO_SUPPLY_IND, Connector_JST:JST_XH_B2B-XH-A_1x02_P2.50mm_Vertical, symbol Device:LED_Small
- added D11: 5V_SUPPLY, Connector_JST:JST_XH_B2B-XH-A_1x02_P2.50mm_Vertical, symbol Device:LED_Small
- added H6: MountingHole, MountingHole:MountingHole_3.2mm_M3, symbol Mechanical:MountingHole
- added Q7: MJD45H11T4G, SamacSys_Parts:MJD45H11AJ, symbol Simulation_SPICE:PNP
- added Q8: MJD44H11T4G, SamacSys_Parts:MJD44H11AJ, symbol Simulation_SPICE:NPN
- added R28, R29: 0, Resistor_SMD:R_0805_2012Metric, symbol Device:R_Small_US
- added R30, R31, R32, R33: 5, Resistor_SMD:R_0805_2012Metric, symbol Device:R_Small_US
- added R34, R35: 10k, Resistor_SMD:R_0805_2012Metric, symbol Device:R_Small_US
- added RV2, RV3: 100k, Potentiometer_THT:Potentiometer_Bourns_3266W_Vertical, symbol Device:R_Potentiometer_US
- added TP1: CH2_OUTPUT, TestPoint:TestPoint_Pad_D1.0mm, symbol Connector:TestPoint
- added TP10: CH3_OPA_OUT, TestPoint:TestPoint_Pad_D1.0mm, symbol Connector:TestPoint
- added TP11: CH2_OPA_OUT, TestPoint:TestPoint_Pad_D1.0mm, symbol Connector:TestPoint
- added TP12: CH1_OPA_OUT, TestPoint:TestPoint_Pad_D1.0mm, symbol Connector:TestPoint
- added TP13: 60V_TEST, TestPoint:TestPoint_Pad_D1.0mm, symbol Connector:TestPoint
- added TP14: 5V_TEST, TestPoint:TestPoint_Pad_D1.0mm, symbol Connector:TestPoint
- added TP15: 6V2_TEST, TestPoint:TestPoint_Pad_D1.0mm, symbol Connector:TestPoint
- added TP16, TP17, TP18, TP19, TP21, TP22, TP23, TP24, TP25: GNDV_TESTPOINT, TestPoint:TestPoint_Pad_D1.0mm, symbol Connector:TestPoint
- added TP2: CH1_OUTPUT, TestPoint:TestPoint_Pad_D1.0mm, symbol Connector:TestPoint
- added TP20: 5V_VREF_TEST, TestPoint:TestPoint_Pad_D1.0mm, symbol Connector:TestPoint
- added TP26: SCLK_TP, TestPoint:TestPoint_Pad_D1.0mm, symbol Connector:TestPoint
- added TP27: DIN_TP, TestPoint:TestPoint_Pad_D1.0mm, symbol Connector:TestPoint
- added TP28: L_SCLK_TP, TestPoint:TestPoint_Pad_D1.0mm, symbol Connector:TestPoint
- added TP29: L_DIN_TP, TestPoint:TestPoint_Pad_D1.0mm, symbol Connector:TestPoint
- added TP3: CH3_OUTPUT, TestPoint:TestPoint_Pad_D1.0mm, symbol Connector:TestPoint
- added TP30: XTAL_0_TP, TestPoint:TestPoint_Pad_D1.0mm, symbol Connector:TestPoint
- added TP31: XTAL_1_TP, TestPoint:TestPoint_Pad_D1.0mm, symbol Connector:TestPoint
- added TP32, TP33: GND_TP, TestPoint:TestPoint_Pad_D1.0mm, symbol Connector:TestPoint
- added TP4: CH4_OUTPUT, TestPoint:TestPoint_Pad_D1.0mm, symbol Connector:TestPoint
- added TP5: CH4_AN_IN, TestPoint:TestPoint_Pad_D1.0mm, symbol Connector:TestPoint
- added TP6: CH3_AN_IN, TestPoint:TestPoint_Pad_D1.0mm, symbol Connector:TestPoint
- added TP7: CH2_AN_IN, TestPoint:TestPoint_Pad_D1.0mm, symbol Connector:TestPoint
- added TP8: CH1_AN_IN, TestPoint:TestPoint_Pad_D1.0mm, symbol Connector:TestPoint
- added TP9: CH4_OPA_OUT, TestPoint:TestPoint_Pad_D1.0mm, symbol Connector:TestPoint
- D1, D2: value BZT52-C5V6 -> BZT52-C6V2
- Q1, Q3, Q5: footprint (none) -> SamacSys_Parts:MJD45H11AJ
- Q10, Q9: footprint (none) -> Package_TO_SOT_SMD:SOT-89-3
- Q11, Q12: footprint (none) -> Package_TO_SOT_SMD:TO-252-2
- Q2, Q4, Q6: footprint (none) -> SamacSys_Parts:MJD44H11AJ
- R1, R10, R11, R12, R13, R14, R15, R16, R19, R2, R20, R21, R22, R23, R24, R25, R26, R27, R3, R4, R5, R6, R7, R8, R9: footprint Capacitor_SMD:C_0805_2012Metric -> Resistor_SMD:R_0805_2012Metric
- RV1: footprint Capacitor_SMD:C_0805_2012Metric -> Potentiometer_THT:Potentiometer_Bourns_3266W_Vertical
Connections:
- net DIN2 is gone; now on net DIN1: J1.2
- net DIN4 is gone; now on net DIN3: J4.2
- net DO2 is gone; now on net DO1: J1.7
- net DO4 is gone; now on net DO3: J4.7
- net PC13 is gone; now on net BTN1: J10.2 (Pin_2), U4.2 (PC13)
- net PC14 is gone; now on net BTN2: J10.4 (Pin_4), U4.3 (PC14)
- net PC15 is gone; now on net BTN3: J10.6 (Pin_6), U4.4 (PC15)
- net VREF+ is gone; now on net +3V3: C7.2, U4.20 (VREF+)
- net +3V3: now also J10.12 (Pin_12), C46.1, C47.1; no longer J10.10 (Pin_10)
- net +5V: now also J10.10 (Pin_10), R35.1; no longer J10.12 (Pin_12)
- net +5V_HV: now also C48.1, C49.1, TP14.1
- net +5V_REF: now also TP20.1
- net +60V: now also Q10.2 (C), Q11.2 (D), Q2.2 (C), Q4.2 (C), Q6.2 (C), Q9.2 (C), Q8.2 (C), RV2.1, RV3.1, TP13.1; no longer Q10.1 (C), Q11.1 (D), Q2.1 (C), Q4.1 (C), Q6.1 (C), Q9.1 (C)
- net +60V_IN: now also R34.1
- net BTN1: no longer J10.1 (Pin_1), U4.34 (PA12)
- net BTN2: no longer J10.3 (Pin_3), U4.46 (PB9)
- net BTN3: no longer J10.5 (Pin_5), U4.22 (PB10)
- net BTN4: now also J10.8 (Pin_8), U4.12 (PA4); no longer J10.7 (Pin_7), U4.39 (PA15)
- net CONN_TEST_1_P: now also U4.33 (PA11); no longer U4.30 (PA8)
- net CONN_TEST_2_P: now also U4.32 (PA10); no longer U4.31 (PA9)
- net CONN_TEST_3_P: now also U4.31 (PA9); no longer U4.32 (PA10)
- net CONN_TEST_4_P: now also U4.30 (PA8); no longer U4.33 (PA11)
- net DIN: now also TP27.1
- net GND: now also J6.SH1 (SHIELD), J6.SH2 (SHIELD), J6.SH3 (SHIELD), J6.SH4 (SHIELD), C46.2, C47.2, D11.1 (K), TP32.1, TP33.1; no longer C30.1, C31.1, C32.1, C39.1, J6.S1 (SHIELD)
- net GNDV: now also C30.1, C31.1, C32.1, C39.1, Q1.2 (C), Q3.2 (C), Q5.2 (C), C48.2, C49.2, C51.1, C52.1, C54.1, C56.1, D10.1 (K), Q7.2 (C), RV2.3, RV3.3, TP16.1, TP17.1, TP18.1, TP19.1, TP21.1, TP22.1, TP23.1, TP24.1, TP25.1; no longer Q1.1 (C), Q3.1 (C), Q5.1 (C)
- net PIEZO_CH1_PA: now also R31.1, TP2.1; no longer Q3.3 (E), Q4.3 (E), R10.1, R11.1
- net PIEZO_CH1_SIG: now also TP8.1
- net PIEZO_CH2_PA: now also R30.1, TP1.1; no longer Q1.3 (E), Q2.3 (E), R13.1, R2.1
- net PIEZO_CH2_SIG: now also TP7.1
- net PIEZO_CH3_PA: now also R32.1, TP3.1; no longer R14.1, R6.1
- net PIEZO_CH3_SIG: now also TP6.1
- net PIEZO_CH4_PA: now also R33.1, TP4.1; no longer Q5.3 (E), Q6.3 (E), R15.1, R16.1
- net PIEZO_CH4_SIG: now also TP5.1
- net SCLK: now also TP26.1
- net ~{CS1}: now also U4.18 (PB2); no longer U4.26 (PB12)
- net ~{CS2}: now also U4.46 (PB9); no longer U4.25 (PB11)
- net ~{CS3}: now also U4.39 (PA15); no longer U4.18 (PB2)
- net ~{CS4}: now also U4.26 (PB12); no longer U4.17 (PB1)
- net at R11.2, U5.6: now also Q3.1 (B), Q4.1 (B), TP12.1; no longer Q3.2 (B), Q4.2 (B)
- net at Q12.3 (S): now also Q11.1 (G); no longer Q11.2 (G)
- net at R15.2, U7.6: now also Q7.1 (B), Q8.1 (B), TP9.1; no longer Q5.2 (B), Q6.2 (B)
- net at U1.2 (INA): now also R28.2; no longer U4.12 (PA4)
- net at U4.14 (PA6): now also R29.1; no longer U1.3 (INB)
- net at C1.2, U4.5 (PF0), Y1.2: now also TP30.1
- net at C2.2, U4.6 (PF1), Y1.1: now also TP31.1
- net at JP2.2 (B): now also Q9.1 (E); no longer Q9.3 (E)
- net at R1.1, R2.2, U9.2 (-): now also C54.2, C55.1
- net at R6.2, R7.1, U8.2 (-): now also C52.2, C53.1
- net at D1.1 (K): now also Q9.3 (B), RV2.2; no longer Q9.2 (B)
- net at D2.1 (K): now also Q10.3 (B), RV3.2; no longer Q10.2 (B)
- net at R13.2, U9.6: now also Q1.1 (B), Q2.1 (B), TP11.1; no longer Q1.2 (B), Q2.2 (B)
- net at R12.1, R16.2, U7.2 (-): now also C50.1, C51.2
- net at JP3.1 (A): now also Q10.1 (E); no longer Q10.3 (E)
- net at C19.2, JP3.2 (B), U10.2 (Vin): now also TP15.1
- net at R14.2, U8.6: now also Q5.1 (B), Q6.1 (B), TP10.1
- net at R24.2, R27.2: now also Q12.2 (D); no longer Q12.1 (D)
- net at R4.2, U6.2 (INA): now also TP28.1
- net at D8.1 (K), R23.1, RV1.3: now also Q12.1 (G); no longer Q12.2 (G)
- net at R5.2, U6.3 (INB): now also TP29.1
- net at R10.2, R9.1, U5.2 (-): now also C56.2, C57.1
- net PB0: no longer names the net of U4.16 (PB0)
- net PB0: now also R28.1; no longer J10.8 (Pin_8)
- new net: C57.2, Q3.3 (E), Q4.3 (E), R10.1, R11.1, R31.2
- new net: C55.2, Q1.3 (E), Q2.3 (E), R13.1, R2.1, R30.2
- new net: C50.2, Q7.3 (E), Q8.3 (E), R15.1, R16.1, R33.2
- new net: R29.2, U1.3 (INB)
- new net: C53.2, Q5.3 (E), Q6.3 (E), R14.1, R32.2, R6.1
- new net: D10.2 (A), R34.2
- new net: D11.2 (A), R35.2
- no-connect marks 14 -> 22
Other:
- note added: "Adjust C50,C53,C55,C57 higher if overshoot/oscillation occurs"
- note added: "Adjust R30,R31,R32,R33 higher if overshoot/oscillation occurs. Keep within 10ohm"
- moved on the sheet: C18, C19, C20, C29, C40, C41, C42, C45, D1, D2, D7, D8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
